Commit message: Agrega launc.py nuevos y modificacion de meshes

File: urdf/puzzlebot.urdf.xacro (robot description, xacro)
@@ -10,5 +10,5 @@
       <origin xyz="0 0 0.05" rpy="0 0 0"/>
       <geometry>
-        <mesh filename="package://ServoYSirvo_nav2_puzzlebot/meshes/Puzzlebot_Jetson_Lidar_Edition_Base.stl"/>
+        <mesh filename="package://ServoYSirvo_nav2_puzzlebot/meshes/bases/Puzzlebot_Jetson_Lidar_Edition_Base.stl"/>
       </geometry>
       <material name="gray"/>
@@ -17,5 +17,5 @@
       <origin xyz="0 0 0.05" rpy="0 0 0"/>
       <geometry>
-        <mesh filename="package://ServoYSirvo_nav2_puzzlebot/meshes/Puzzlebot_Jetson_Lidar_Edition_Base.stl"/>
+        <mesh filename="package://ServoYSirvo_nav2_puzzlebot/meshes/bases/Puzzlebot_Jetson_Lidar_Edition_Base.stl"/>
       </geometry>
     </collision>
@@ -32,5 +32,5 @@
       <origin xyz="-0.095 0.0 -0.03" rpy="0 0 0"/>
       <geometry>
-        <mesh filename="package://ServoYSirvo_nav2_puzzlebot/meshes/Puzzlebot_Caster_Wheel.stl"/>
+        <mesh filename="package://ServoYSirvo_nav2_puzzlebot/meshes/wheels/Puzzlebot_Caster_Wheel.stl"/>
       </geometry>
       <material name="gray"/>
@@ -47,5 +47,5 @@
       <origin xyz="0.052 0.095 -0.0025" rpy="0 0 0"/>
       <geometry>
-        <mesh filename="package://ServoYSirvo_nav2_puzzlebot/meshes/Puzzlebot_Wheel.stl"/>
+        <mesh filename="package://ServoYSirvo_nav2_puzzlebot/meshes/wheels/Puzzlebot_Wheel.stl"/>
       </geometry>
       <material name="gray"/>
@@ -63,5 +63,5 @@
       <origin xyz="0.052 -0.095 -0.0025" rpy="0 0 0"/>
       <geometry>
-        <mesh filename="package://ServoYSirvo_nav2_puzzlebot/meshes/Puzzlebot_Wheel.stl"/>
+        <mesh filename="package://ServoYSirvo_nav2_puzzlebot/meshes/wheels/Puzzlebot_Wheel.stl"/>
       </geometry>
       <material name="gray"/>
